File: EAGLE/vr01/vr01-revA.sch (EAGLE design)
At the start: 11 parts, among them J1 CX60-24S-UNIT, SW1 SPST_TACT-KMR2, SW2 SPST_TACT-KMR2, U1 ESP32-C6-MINI-1, U2 AP2112K-3.3

Commit message: .
Parts:
- removed LK-USB07: CASE-LK-USB07-OPEN-ENDS, vr01-footprints:CASE-LK-USB07-OPEN-ENDS
- removed SW1, SW2: SPST_TACT-KMR2, adafruit:SPST_TACT-KMR2
- removed U$3: TRINKEYDRILLS, __vr01-footprints:TRINKEYDRILLS
- removed USBSEL: TS3USB221A-Q1, ts_kb_mcu:TS3USB221A-Q1
- added C2, C3, C6: 100nF, rcl:C-EUC0402K
- added C4, C5: 4.3pF, rcl:C-EUC0402K
- added C7: 10uF, rcl:C-EUC0402K
- added D1: NSR0320, adafruit:DIODESOD-323F
- added J2: (no value), Seeeduino-XIAO-footprint-eagle:HEADER-7P-HALF-HOLE-2.54
- added J3, J4, J5, J6, J7, J8: (no value), SparkFun-Connectors:CONN_07
- added L1: BEAD, SparkFun-Coils:FERRITE_BEAD
- added R1, R2: 10R, rcl:R-EU_R0402
- added R10, R15, R8: 10K, rcl:R-EU_R0603
- added R11, R12, R7, R9: (no value), rcl:R-EU_R0603
- added R13, R14: 5.1K, rcl:R-EU_R0603
- added R3: FUSE, microbuilder:RESISTOR0805_NOOUTLINE
- added R4, R5: 5.1K, rcl:R-EU_R0402
- added R6: 10K, rcl:R-EU_R0402
- added TP1, TP2: TEST-POINT.4RN, tecsmith_keyboards:TEST-POINT.4RN
- added U$11, U$12: MX-5-PIN-HOTSWAP-VIANO-SILK, tecsmith_keyboards:MX-5-PIN-HOTSWAP-VIANO-SILK
- added U$13, U$14: SK6812-MINI-ESK6812MINI-E, tecsmith_keyboards:SK6812-MINI-ESK6812MINI-E
- added U$16, U$19: MX-FPRINT-100U-DOC, tecsmith_keyboards:MX-FPRINT-100U-DOC
- added U$17, U$18: 74AHCT1G125GW, tecsmith_keyboards:74AHCT1G125GW
- added U$21: HE-2-PIN-HOTSWAP, tecsmith_keyboards:HE-2-PIN-HOTSWAP
- added X1: (no value), tecsmith_keyboards:USB_C
- added Y1: 3.2768KHz, OPL_Crystal Oscillator:SMD-CRYSTAL-32.768KHZ-12.5PF-20PPM-90K(2P-L2.0X1.2MM)
- C1: value 10uF -> 100nF; device microbuilder:CAP_CERAMIC0805-NOOUTLINE -> rcl:C-EUC0402K
- C8: device microbuilder:CAP_CERAMIC0805-NOOUTLINE -> rcl:C-EUC0402K
- J1: value CX60-24S-UNIT -> (none); device vr01-footprints:CX60-24S-UNIT -> Seeeduino-XIAO-footprint-eagle:HEADER-7P-HALF-HOLE-2.54
- U1: value ESP32-C6-MINI-1 -> EC11E15244B2; device vr01-footprints:ESP32-C6-MINI-1 -> tecsmith_keyboards:EC11E15244B2
Connections:
- removed net +3V3: C8.1, U2.OUT
- removed net +5V: C1.1, U2.EN, U2.IN
- removed net GND1: C1.2, C8.2, U2.GND
- removed net GND2: USBSEL.GND
- removed net USB1_N: USBSEL.1D-
- removed net USB1_P: USBSEL.1D+
- removed net USB2_N: USBSEL.2D-
- removed net USB2_P: USBSEL.2D+
- new net !RST: C6.1, STM32G$1.!RST, TP1.1
- new net A0D0: J1.1, STM32G$1.PA0
- new net A1D1: J1.2, STM32G$1.PA1
- new net A2D2: J1.3, STM32G$1.PA2
- new net A3D3: J1.4, STM32G$1.PA3
- new net BOOT0: R6.2, STM32G$1.BOOT0
- new net ENC1: J7.7, R13.1, U1.A
- new net ENC2: J8.1, R14.1, U1.B
- new net GND: C1.2, C2.2, C3.2, C4.2, C5.2, C6.2, C7.2, C8.2, J2.6, J4.6, J6.6, J8.6, R10.1, R15.1, R4.2, R5.2, R6.1, R8.1, STM32G$2.VSS, STM32G$2.VSS2/PB2, TP2.1, U$13.GND, U$14.GND, U$17.!OE, U$17.3_GND, U$18.!OE, U$18.3_GND, U$21.GND, U1.C, U2.GND, X1.GND, X1.SHIELD
- new net HE1: J5.3, U$21.OUT
- new net LED: STM32G$1.PB3
- new net MISO: J2.3, STM32G$1.PA6
- new net MOSI: J2.4, STM32G$1.PA7
- new net N$1: C1.1, L1.2, STM32G$2.VDDA
- new net N$10: R9.1, U$13.DIN
- new net N$11: R9.2, U$17.Y_DOUT
- new net N$12: R12.1, U$14.DIN
- new net N$13: R12.2, U$18.Y_DOUT
- new net N$14: R11.1, U$18.A_DIN
- new net N$15: R7.1, U$17.A_DIN
- new net N$2: C4.1, STM32G$1.PF0-OSC_IN, Y1.2
- new net N$3: C5.1, STM32G$1.PF1-OSC_OUT, Y1.1
- new net N$4: R4.1, X1.CC1
- new net N$5: R5.1, X1.CC2
- new net N$6: C7.1, D1.C, U2.EN, U2.IN
- new net N$7: D1.A, R3.2
- new net N$8: R1.1, X1.D+1, X1.D+2
- new net N$9: R2.1, X1.D-1, X1.D-2
- new net NSS: STM32G$1.PA4
- new net RCC: STM32G$1.PA8
- new net RGB: J3.1, R11.2, R7.2
- new net RX: J2.1, STM32G$1.PB7
- new net SCK: J2.2, STM32G$1.PA5
- new net SCL: J1.6, STM32G$1.PB6
- new net SDA: J1.5, STM32G$1.PA10
- new net SW1: J3.4, R10.2, R8.2, U$11.1, U$12.2
- new net SW2: J7.2, R15.2, U1.E
- new net SWCLK: STM32G$1.PA14
- new net SWDIO: STM32G$1.PA13
- new net TX: J1.7, STM32G$1.PA9
- new net USB_N: R2.2, STM32G$1.PA11
- new net USB_P: R1.2, STM32G$1.PA12
- new net VCC3: C2.1, C3.1, C8.1, J2.5, J4.5, J6.5, J8.5, L1.1, R13.2, R14.2, STM32G$2.VDD, STM32G$2.VDDIO2, U$11.2, U$12.1, U$21.VDD, U1.D, U2.OUT
- new net VCC5: J2.7, J4.7, J6.7, J8.7, R3.1, U$13.VDD, U$14.VDD, U$17.5_VCC, U$18.5_VCC, X1.VBUS
Other:
- note added: "EC11 Rotary Encoder"
- note added: "Hall Effect Switch"
- note added: "MX Mechanical Swith"
- note added: "RESET"
- note added: "STM32F042 "XIAO" Footprint"
- moved on the sheet: C1, C8, STM32G$1, U2
