File: EAGLE/vr01/vr01-revC.brd (EAGLE design)
At the start: 66 x 43.2 mm, 46 parts, among them SW1A MX-5-PIN-HOTSWAP-VIANO-SILK, SW1B MX-5-PIN-HOTSWAP-VIANO-SILK, U1 EC11E15244B2

Commit message: .
Parts:
- added J10, J11: QWIIC_RIGHT_ANGLE, tecsmith_custom_nick_nacks:JST04_1MM_RA
- added U$2, U$4, U$5: FIDUCIAL, tecsmith_custom_nick_nacks:FIDUCIAL
Connections:
- new net SCL: J10.4, J11.4, J5.6
- new net SDA: J10.3, J11.3, J5.5
- net GND: now also J10.1, J11.1
- net VCC3: now also J10.2, J11.2
Routing:
- net VCC3: track 80.3 -> 103.7 mm, vias 4 -> 5
- net SDA: track 0.00 -> 14.2 mm
- net SCL: track 0.00 -> 12.3 mm
- net RGB: track 15.7 -> 15.2 mm, vias 1 -> 2
- net GND: vias 61 -> 65
Other:
- board text added: "(c) 2024"
- board text added: "DRV5056"
- board text added: "EC11"
- board text added: "MX"
- board text added: "Tecsmith VR01"
- board text added: "Vino Rodrigues"
- board text added: "XIAO ESP32"
