File: EAGLE/vr01/vr01-revC.sch (EAGLE design)
At the start: 46 parts, among them SW1A MX-5-PIN-HOTSWAP-VIANO-SILK, SW1B MX-5-PIN-HOTSWAP-VIANO-SILK, U1 EC11E15244B2

Commit message: .
Parts:
- added J10, J11: QWIIC_RIGHT_ANGLE, tecsmith_custom_nick_nacks:QWIIC_CONNECTORJS-1MM
- added U$2, U$4, U$5: FIDUCIAL, tecsmith_custom_nick_nacks:FIDUCIAL
Connections:
- new net SCL: J10.4, J11.4, J5.6
- new net SDA: J10.3, J11.3, J5.5
- net GND: now also J10.1, J11.1
- net VCC3: now also J10.2, J11.2
Changed lines of the file:
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@@
 <part name="C6A" library="rcl" library_urn="urn:adsk.eagle:library:334" deviceset="C-EU" device="C0603" package3d_urn="urn:adsk.eagle:package:23616/2" value="0.1uF"/>
 <part name="GND6" library="tecsmith_custom_nick_nacks" deviceset="GND" device=""/>
+<part name="U$2" library="tecsmith_custom_nick_nacks" deviceset="FIDUCIAL" device=""/>
+<part name="U$4" library="tecsmith_custom_nick_nacks" deviceset="FIDUCIAL" device=""/>
+<part name="U$5" library="tecsmith_custom_nick_nacks" deviceset="FIDUCIAL" device=""/>
+<part name="J10" library="tecsmith_custom_nick_nacks" deviceset="QWIIC_CONNECTOR" device="JS-1MM" value="QWIIC_RIGHT_ANGLE"/>
+<part name="J11" library="tecsmith_custom_nick_nacks" deviceset="QWIIC_CONNECTOR" device="JS-1MM" value="QWIIC_RIGHT_ANGLE"/>
+<part name="U$6" library="tecsmith_custom_nick_nacks" deviceset="3V3" device=""/>
+<part name="U$10" library="tecsmith_custom_nick_nacks" deviceset="3V3" device=""/>
+<part name="GND7" library="tecsmith_custom_nick_nacks" deviceset="GND" device=""/>
+<part name="GND8" library="tecsmith_custom_nick_nacks" deviceset="GND" device=""/>
 </parts>
 <sheets>
@@
 <attribute name="VALUE" x="190.5" y="79.248" size="1.778" layer="96" align="top-center"/>
 </instance>
+<instance part="U$2" gate="G$1" x="157.48" y="5.08" smashed="yes"/>
+<instance part="U$4" gate="G$1" x="152.4" y="5.08" smashed="yes"/>
+<instance part="U$5" gate="G$1" x="147.32" y="5.08" smashed="yes"/>
+<instance part="J10" gate="G$1" x="175.26" y="106.68" smashed="yes">
+<attribute name="VALUE" x="170.18" y="101.346" size="1.778" layer="96" font="vector" align="top-left"/>
+<attribute name="NAME" x="170.18" y="114.554" size="1.778" layer="95" font="vector"/>
+</instance>
+<instance part="J11" gate="G$1" x="203.2" y="106.68" smashed="yes">
+<attribute name="VALUE" x="198.12" y="101.346" size="1.778" layer="96" font="vector" align="top-left"/>
+<attribute name="NAME" x="198.12" y="114.554" size="1.778" layer="95" font="vector"/>
+</instance>
+<instance part="U$6" gate="G$1" x="185.42" y="106.68" smashed="yes" rot="R270">
+<attribute name="VALUE" x="190.5" y="106.68" size="1.778" layer="96" rot="R270" align="bottom-center"/>
+</instance>
+<instance part="U$10" gate="G$1" x="213.36" y="106.68" smashed="yes" rot="R270">
+<attribute name="VALUE" x="218.44" y="106.68" size="1.778" layer="96" rot="R270" align="bottom-center"/>
+</instance>
+<instance part="GND7" gate="1" x="185.42" y="104.14" smashed="yes" rot="R90">
+<attribute name="VALUE" x="189.992" y="104.14" size="1.778" layer="96" rot="R90" align="top-center"/>
+</instance>
+<instance part="GND8" gate="1" x="213.36" y="104.14" smashed="yes" rot="R90">
+<attribute name="VALUE" x="217.932" y="104.14" size="1.778" layer="96" rot="R90" align="top-center"/>
+</instance>
 </instances>
 <busses>
@@
 <wire x1="182.88" y1="149.86" x2="182.88" y2="147.32" width="0.1524" layer="91"/>
 <junction x="182.88" y="147.32"/>
+</segment>
+<segment>
+<pinref part="J10" gate="G$1" pin="2"/>
+<wire x1="182.88" y1="106.68" x2="185.42" y2="106.68" width="0.1524" layer="91"/>
+<pinref part="U$6" gate="G$1" pin="VCC3"/>
+</segment>
+<segment>
+<pinref part="J11" gate="G$1" pin="2"/>
+<wire x1="210.82" y1="106.68" x2="213.36" y2="106.68" width="0.1524" layer="91"/>
+<pinref part="U$10" gate="G$1" pin="VCC3"/>
 </segment>
 </net>
@@
 <pinref part="GND6" gate="1" pin="GND"/>
 <wire x1="190.5" y1="86.36" x2="190.5" y2="83.82" width="0.1524" layer="91"/>
+</segment>
+<segment>
+<pinref part="J10" gate="G$1" pin="1"/>
+<wire x1="182.88" y1="104.14" x2="185.42" y2="104.14" width="0.1524" layer="91"/>
+<pinref part="GND7" gate="1" pin="GND"/>
+</segment>
+<segment>
+<pinref part="J11" gate="G$1" pin="1"/>
+<wire x1="210.82" y1="104.14" x2="213.36" y2="104.14" width="0.1524" layer="91"/>
+<pinref part="GND8" gate="1" pin="GND"/>
 </segment>
 </net>
@@
 </segment>
 </net>
+<net name="SCL" class="0">
+<segment>
+<pinref part="J5" gate="J1" pin="6"/>
+<wire x1="236.22" y1="147.32" x2="233.68" y2="147.32" width="0.1524" layer="91"/>
+<label x="231.14" y="144.78" size="1.778" layer="95" rot="R180" xref="yes"/>
+<wire x1="233.68" y1="147.32" x2="233.68" y2="144.78" width="0.1524" layer="91"/>
+<wire x1="233.68" y1="144.78" x2="231.14" y2="144.78" width="0.1524" layer="91"/>
+</segment>
+<segment>
+<pinref part="J10" gate="G$1" pin="4"/>
+<wire x1="182.88" y1="111.76" x2="185.42" y2="111.76" width="0.1524" layer="91"/>
+<label x="185.42" y="111.76" size="1.4224" layer="95" xref="yes"/>
+</segment>
+<segment>
+<pinref part="J11" gate="G$1" pin="4"/>
+<wire x1="210.82" y1="111.76" x2="213.36" y2="111.76" width="0.1524" layer="91"/>
+<label x="213.36" y="111.76" size="1.4224" layer="95" xref="yes"/>
+</segment>
+</net>
+<net name="SDA" class="0">
+<segment>
+<pinref part="J5" gate="J1" pin="5"/>
+<wire x1="236.22" y1="149.86" x2="231.14" y2="149.86" width="0.1524" layer="91"/>
+<label x="231.14" y="149.86" size="1.778" layer="95" rot="R180" xref="yes"/>
+</segment>
+<segment>
+<pinref part="J10" gate="G$1" pin="3"/>
+<wire x1="182.88" y1="109.22" x2="185.42" y2="109.22" width="0.1524" layer="91"/>
+<label x="185.42" y="109.22" size="1.4224" layer="95" xref="yes"/>
+</segment>
+<segment>
+<pinref part="J11" gate="G$1" pin="3"/>
+<wire x1="210.82" y1="109.22" x2="213.36" y2="109.22" width="0.1524" layer="91"/>
+<label x="213.36" y="109.22" size="1.4224" layer="95" xref="yes"/>
+</segment>
+</net>
