File: KiCAD/sr01/sr01.kicad_pcb (KiCad board)
At the start: 2 copper layers, 67 x 38 mm, 54 parts, among them J1 Conn_01x02, J2 Conn_01x01, J3 Conn_01x01, J4 Conn_01x01, SW3 EC11, U4 SW_DRV5056

Commit message: add EC switch
Parts:
- added C8: 0.1uF, Capacitor_SMD:C_0603_1608Metric, B.Cu at (76.0, 66.5)
- added C9: 220p, Capacitor_SMD:C_0603_1608Metric, B.Cu at (83.0, 73.0)
- added J5: ~, Connector_JST:JST_SH_SM04B-SRSS-TB_1x04-1MP_P1.00mm_Horizontal, B.Cu at (69.0, 70.0)
- added R11: 100K, Resistor_SMD:R_0603_1608Metric, B.Cu at (74.0, 74.0)
- added R12: DNP, Resistor_SMD:R_0603_1608Metric, B.Cu at (74.0, 75.5)
- added R13: 1K, Resistor_SMD:R_0603_1608Metric, B.Cu at (77.5, 74.0)
- added R14: 100K, Resistor_SMD:R_0603_1608Metric, B.Cu at (83.0, 74.5)
- added R15: 100R, Resistor_SMD:R_0603_1608Metric, B.Cu at (83.0, 65.5)
- added REF**: Drawing_EC_1U, ts-keyboard-ec-lib:Drawing_EC_1U, F.Cu at (91.0, 70.0)
- added REF**: PlaceCut_MX_1U_Alt, ts-keyboard-lib:PlaceCut_MX_1U_Alt, F.Cu at (123.0, 50.0)
- added REF**: Value, ts-keyboard-ec-lib:PlaceCut_EC_DynaCap_1U, F.Cu at (120.0, 70.0)
- added TP1: ~, TestPoint:TestPoint_Keystone_5000-5004_Miniature, F.Cu at (103.0, 73.5)
- added TP2: ~, TestPoint:TestPoint_Keystone_5000-5004_Miniature, F.Cu at (103.0, 66.5)
- added TP3: ~, TestPoint:TestPoint_Keystone_5000-5004_Miniature, F.Cu at (68.0, 75.5)
- added TP4: ~, TestPoint:TestPoint_Keystone_5000-5004_Miniature, F.Cu at (103.0, 70.0)
- added TP5: ~, TestPoint:TestPoint_Keystone_5000-5004_Miniature, F.Cu at (67.9, 64.5)
- added U5: ~, ts-seeed-xiao-lib:XIAO-Generic-DIP, F.Cu at (77.0, 70.0)
- added U6: ~, ts-keyboard-ec-lib:SW_EC_1U, B.Cu at (91.0, 70.0)
- added U7: OPA350, Package_SO:SOIC-8_3.9x4.9mm_P1.27mm, B.Cu at (76.0, 70.0)
- added mouse-bite-2mm-slot: VAL**, ts-kicad-lib:mouse-bite-2mm-slot, F.Cu at (123.0, 60.0)
- added mouse-bite-2mm-slot: VAL**, ts-kicad-lib:mouse-bite-2mm-slot, F.Cu at (77.0, 60.0)
- added mouse-bite-2mm-slot: VAL**, ts-kicad-lib:mouse-bite-2mm-slot, F.Cu at (105.5, 70.0)
- added mouse-bite-2mm-slot: VAL**, ts-kicad-lib:mouse-bite-2mm-slot, F.Cu at (100.0, 60.0)
Connections:
- net ADC renamed ADC1
Routing:
- net COL: track 0.00 -> 51.3 mm, vias 0 -> 1
- net SCL2: track 0.00 -> 23.8 mm, vias 0 -> 1
- net ROW: track 0.00 -> 23.4 mm
- net +3V3: track 74.0 -> 97.1 mm
- net SDA2: track 0.00 -> 22.5 mm, vias 0 -> 2
- net ADC2: track 0.00 -> 17.5 mm
- net Net-(U7-In-): track 0.00 -> 10.3 mm
- net GND: track 23.9 -> 32.8 mm, vias 63 -> 80
- net Net-(R15-Pad2): track 0.00 -> 8.72 mm
- net +5V: track 145.9 -> 147.2 mm
- added copper zone on B.Cu, net +3V3
Other:
- board size 67 x 38 mm -> 67 x 58 mm
