File: KiCAD/sr01/sr01.kicad_sch (KiCad schematic)
At the start: 46 parts, among them J1 Conn_01x02, J2 Conn_01x01, J3 Conn_01x01, J4 Conn_01x01, SW3 EC11, U4 SW_DRV5056

Commit message: add EC switch
Parts:
- added C8: 0.1uF, Capacitor_SMD:C_0603_1608Metric, symbol ts-kicad-lib:C
- added C9: 220p, Capacitor_SMD:C_0603_1608Metric, symbol ts-kicad-lib:C
- added J5: (no value), Connector_JST:JST_SH_SM04B-SRSS-TB_1x04-1MP_P1.00mm_Horizontal, symbol ts-kicad-lib:QWIIC
- added R11, R14: 100K, Resistor_SMD:R_0603_1608Metric, symbol ts-kicad-lib:R
- added R12: DNP, Resistor_SMD:R_0603_1608Metric, symbol ts-kicad-lib:R
- added R13: 1K, Resistor_SMD:R_0603_1608Metric, symbol ts-kicad-lib:R
- added R15: 100R, Resistor_SMD:R_0603_1608Metric, symbol ts-kicad-lib:R
- added TP1, TP2, TP3, TP4, TP5: (no value), TestPoint:TestPoint_Keystone_5000-5004_Miniature, symbol ts-kicad-lib:TEST_POINT
- added U5: (no value), ts-seeed-xiao-lib:XIAO-Generic-DIP, symbol ts-seeed-xiao-lib:XIAO-HEADER
- added U6: (no value), ts-keyboard-ec-lib:SW_EC_1U, symbol ts-keyboard-ec-lib:SW_EC_DynaCap
- added U7: OPA350, Package_SO:SOIC-8_3.9x4.9mm_P1.27mm, symbol ts-keyboard-ec-lib:OPA350
- U1, U2, U3: footprint (none) -> ts-seeed-xiao-lib:XIAO-Generic-DIP
Connections:
- net +3V3: now also C8.2, J5.2, TP5.1, U5.12 (3v3), U7.7 (V+)
- net +5V: now also U5.14 (5V)
- net GND: now also C8.1, C9.1, J5.1, J5.MP, R13.2, R14.2, TP4.1, U5.13 (GND), U6.3, U7.4 (V-)
- net ADC renamed ADC1
- new net: R11.2, R12.2, R13.1, U7.2 (In-)
- new net: U7.1 (N/C), U7.5 (N/C), U7.8 (N/C)
- new net: R15.2, U6.2
- new net ADC2: R11.1, R12.1, TP3.1, U5.1 (io0), U7.6 (Out)
- new net COL: C9.2, R14.1, TP1.1, U5.3 (io2), U5.4 (io3), U6.1, U7.3 (In+)
- new net ROW: R15.1, TP2.1
- new net SCL2: J5.4, U5.6 (SCL)
- new net SDA2: J5.3, U5.5 (SDA)
Other:
- note added: "EC Switch"
- note removed: "Switch Plate"
